File: sd2iec_sd_long.brd (EAGLE design)
At the start: 52.5 x 36.1 mm, 41 parts, among them IC1 MEGA644P, IC3 LP2950_3.0, Q1 8,0 MHz, SW1 Disk Next, SW2 Reset, SW3 Disk Prev, T2 IRLML2402, T3 IRLML2402, T4 IRLML2402

Commit message: Add files via upload
Parts:
- moved X1 0.56 mm to (1.27, 3.17)
- moved U$7 0.22 mm to (1.75, 24.1)
- moved IC3 0.08 mm to (21.6, 7.62)
Routing:
- net +5V: track 15.4 -> 31.3 mm, vias 0 -> 1
- net WP: track 59.5 -> 66.4 mm
- net GND: track 13.4 -> 6.73 mm, vias 11 -> 20
- net /RESET: track 27.3 -> 29.5 mm
- net DISKPREV: track 13.4 -> 15.0 mm
- net N$25: track 9.39 -> 10.8 mm
- net IEC_ATN: track 16.3 -> 17.3 mm
- net MISO: track 26.1 -> 27.0 mm
- net IEC_DATA: track 10.1 -> 10.9 mm
- net 3V0: track 59.7 -> 60.2 mm
- net IEC_CLK: track 9.22 -> 9.79 mm
Other:
- board size 52.5 x 36.1 mm -> 53.4 x 36.7 mm

Commit message: Add files via upload
Parts:
- moved R2 2.46 mm to (6.43, 4.44)
- moved R3 2.07 mm to (9.60, 4.84)
- moved R4 1.99 mm to (12.5, 4.84)
- moved IC1 1.83 mm to (7.94, 15.8)
- moved U$7 0.51 mm to (1.43, 23.7)
- moved R15 0.16 mm to (6.43, 10.0)
Routing:
- net WP: track 66.4 -> 44.3 mm, vias 0 -> 2
- net N$17: track 11.9 -> 22.6 mm
- net +5V: track 31.3 -> 21.9 mm, vias 1 -> 0
- net MISO: track 27.0 -> 21.1 mm, vias 0 -> 1
- net MOSI: track 18.6 -> 23.9 mm
- net GND: track 6.73 -> 2.63 mm, vias 20 -> 21
- net CS: track 29.3 -> 26.9 mm
- net SCK: track 21.2 -> 19.1 mm, vias 2 -> 1
- net N$20: track 11.0 -> 8.92 mm
- net PC0: track 8.83 -> 10.9 mm
- net 3V0: track 60.2 -> 58.2 mm
- net CLK: track 6.75 -> 8.76 mm
- net IEC_ATN: track 17.3 -> 19.3 mm
- net ATN: track 12.8 -> 14.8 mm
- net PC1: track 3.14 -> 4.94 mm
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